File: CircuitBoard/CircuitBoard.sch (KiCad schematic (older format))
At the start: 12 parts

Commit message: added circuit board
Parts:
- added U?: DOIT-ESP32-DEVKIT-V1, symbol doit-esp32-devkit-v1:DOIT-ESP32-DEVKIT-V1
Changed lines of the file:
@@
 Wire Wire Line
 	2950 1950 3700 1950
+$Comp
+L doit-esp32-devkit-v1:DOIT-ESP32-DEVKIT-V1 U?
+U 1 1 61730A6B
+P 1700 3900
+F 0 "U?" H 1675 4465 50  0000 C CNN
+F 1 "DOIT-ESP32-DEVKIT-V1" H 1675 4374 50  0000 C CNN
+F 2 "" H 1650 4350 50  0001 C CNN
+F 3 "" H 1650 4350 50  0001 C CNN
+	1    1700 3900
+	1    0    0    -1
+$EndComp
 $EndSCHEMATC

Commit message: Added assignment3 documentation folder
Parts:
- added U?: DHT11, Sensor:Aosong_DHT11_5.5x12.0_P2.54mm, symbol Sensor:DHT11
Changed lines of the file:
@@
+	1    0    0    -1
+$EndComp
+$Comp
+L Sensor:DHT11 U?
+U 1 1 61734C4D
+P 3800 4950
+F 0 "U?" H 3556 4996 50  0000 R CNN
+F 1 "DHT11" H 3556 4905 50  0000 R CNN
+F 2 "Sensor:Aosong_DHT11_5.5x12.0_P2.54mm" H 3800 4550 50  0001 C CNN
+F 3 "http://akizukidenshi.com/download/ds/aosong/DHT11.pdf" H 3950 5200 50  0001 C CNN
+	1    3800 4950
 	1    0    0    -1
 $EndComp

Commit message: circuit board update
Parts:
- removed U?: DOIT-ESP32-DEVKIT-V1, symbol doit-esp32-devkit-v1:DOIT-ESP32-DEVKIT-V1
- added R5: 4.7K, symbol Device:R_US
- R1, R2, R3, R4: renamed from 500ohm; value R_US -> 500
Connections:
- net GNDREF: now also U?.4 (GND)
- net VCC: now also U?.1 (VCC), R5.2
- net at U?.2 (IO): now also R5.1
Other:
- moved on the sheet: 100nF, D?, J?, M?, R1, R2, R3, R4, U?
